File: CoCoProtoBoard.kicad_pcb (KiCad board)
At the start: 2 copper layers, 100 x 96 mm, 865 parts, among them P1 CocoEdgeConnector, P10 Power Bus, P2 Coco Data, P3 Coco Address, P4 Coco Signals

Commit message: a little cleanup and new Gerbers
Parts:
- removed ?: , 
- removed the REF** at (123.8, 62.1)
- added C1: 100uF, Capacitor_THT:C_Radial_D6.3mm_H7.0mm_P2.50mm, F.Cu at (126.4, 62.1)
