File: CoCoProtoBoard.kicad_sch (KiCad schematic)
At the start: 6 parts, among them P1 CocoEdgeConnector, P10 Power Bus, P2 Coco Data, P3 Coco Address, P4 Coco Signals

Commit message: a little cleanup and new Gerbers
Parts:
- C1: footprint Capacitors_ThroughHole:C_Radial_D7.5_L11.2_P2.5 -> Capacitor_THT:C_Radial_D6.3mm_H7.0mm_P2.50mm; symbol Device:CP -> Device:C
- P1: footprint 00_Custom:CocoCardEdge -> CoCoProtoBoard:CocoCardEdge; symbol 00_Custom:COCO_EDGE_CONNECTOR -> CocoProtoBoard_Library:COCO_EDGE_CONNECTOR
- P10: footprint Housings_DIP:DIP-16_W7.62mm -> CoCoProtoBoard:DIP-61_W300mm
- P2: footprint Housings_DIP:DIP-16_W7.62mm -> CoCoProtoBoard:DIP-16_W7.62mm
- P3: footprint Housings_DIP:DIP-32_W15.24mm -> CoCoProtoBoard:DIP-32_W15.24mm
- P4: footprint Housings_DIP:DIP-22_W10.16mm -> CoCoProtoBoard:DIP-22_W10.16mm
Changed lines of the file:
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@@
 	)
 	(symbol
-		(lib_id "Device:CP")
+		(lib_id "Device:C")
 		(at 201.93 38.1 0)
 		(unit 1)
@@
 			)
 		)
-		(property "Footprint" "Capacitors_ThroughHole:C_Radial_D7.5_L11.2_P2.5"
+		(property "Footprint" "Capacitor_THT:C_Radial_D6.3mm_H7.0mm_P2.50mm"
 			(at 202.8952 41.91 0)
 			(effects
@@
 			)
 		)
-		(property "Datasheet" ""
+		(property "Datasheet" "~"
 			(at 201.93 38.1 0)
 			(effects
@@
 					(size 1.27 1.27)
 				)
-			)
-		)
-		(property "Description" ""
+				(hide yes)
+			)
+		)
+		(property "Description" "Unpolarized capacitor"
 			(at 201.93 38.1 0)
 			(effects
@@
 					(size 1.27 1.27)
 				)
+				(hide yes)
 			)
 		)
@@
 	)
 	(symbol
-		(lib_id "00_Custom:COCO_EDGE_CONNECTOR")
+		(lib_id "CocoProtoBoard_Library:COCO_EDGE_CONNECTOR")
 		(at 20.32 72.39 0)
 		(unit 1)
@@
 			)
 		)
-		(property "Footprint" "00_Custom:CocoCardEdge"
+		(property "Footprint" "CoCoProtoBoard:CocoCardEdge"
 			(at 17.145 72.39 0)
 			(effects
@@
 			)
 		)
-		(property "Footprint" "Housings_DIP:DIP-32_W15.24mm"
+		(property "Footprint" "CoCoProtoBoard:DIP-32_W15.24mm"
 			(at 99.06 114.3 0)
 			(effects
@@
 			)
 		)
-		(property "Footprint" "Housings_DIP:DIP-16_W7.62mm"
+		(property "Footprint" "CoCoProtoBoard:DIP-16_W7.62mm"
 			(at 99.06 71.12 0)
 			(effects
@@
 			)
 		)
-		(property "Footprint" "Housings_DIP:DIP-22_W10.16mm"
+		(property "Footprint" "CoCoProtoBoard:DIP-22_W10.16mm"
 			(at 99.06 170.18 0)
 			(effects
@@
 			)
 		)
-		(property "Footprint" "Housings_DIP:DIP-16_W7.62mm"
+		(property "Footprint" "CoCoProtoBoard:DIP-61_W300mm"
 			(at 222.25 8.89 0)
 			(effects
